File: IR coffee thermometer.kicad_sch (KiCad schematic)
At the start: 37 parts, among them J2 USB_C_Receptacle_USB2.0_16P, U1 ESP32-C3FH4, U3 AMS1117, X1 40MHz, 15pF

Commit message: basic layout
Parts:
- added U2: (no value), MyLib:MLX90614, symbol 0_MyLib:MLX90614
- J2: footprint Connector_USB:USB_C_Receptacle_HRO_TYPE-C-31-M-12 -> MyLib:USB_C_Receptacle_HRO_TYPE-C-31-M-12
Changed lines of the file:
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@@
 			)
 		)
-		(property "Footprint" "Connector_USB:USB_C_Receptacle_HRO_TYPE-C-31-M-12"
+		(property "Footprint" "MyLib:USB_C_Receptacle_HRO_TYPE-C-31-M-12"
 			(at 62.23 97.79 0)
 			(hide yes)
@@
 					(unit 1)
 				)
+			)
+		)
+	)
+	(symbol
+		(lib_id "0_MyLib:MLX90614")
+		(at 236.22 132.08 0)
+		(unit 1)
+		(body_style 1)
+		(exclude_from_sim no)
+		(in_bom yes)
+		(on_board yes)
+		(in_pos_files yes)
+		(dnp no)
+		(fields_autoplaced yes)
+		(property "Reference" "U2"
+			(at 247.015 127 0)
+			(show_name no)
+			(do_not_autoplace no)
+			(effects
+				(font
+					(size 1.27 1.27)
+				)
+			)
+		)
+		(property "Value" ""
+			(at 236.22 132.08 0)
+			(show_name no)
+			(do_not_autoplace no)
+			(effects
+				(font
+					(size 1.27 1.27)
+				)
+			)
+		)
+		(property "Footprint" "MyLib:MLX90614"
+			(at 236.22 132.08 0)
+			(hide yes)
+			(show_name no)
+			(do_not_autoplace no)
+			(effects
+				(font
+					(size 1.27 1.27)
+				)
+			)
+		)
+		(property "Datasheet" ""
+			(at 236.22 132.08 0)
+			(hide yes)
+			(show_name no)
+			(do_not_autoplace no)
+			(effects
+				(font
+					(size 1.27 1.27)
+				)
+			)
+		)
+		(property "Description" ""
+			(at 236.22 132.08 0)
+			(hide yes)
+			(show_name no)
+			(do_not_autoplace no)
+			(effects
+				(font
+					(size 1.27 1.27)
+				)
+			)
+		)
+		(pin "4"
+		)
+		(pin "3"
+		)
+		(pin "4"
+		)
+		(pin "1"
+		)
+		(instances
+			(project "IR coffee thermometer"
+				(path "/ed3d3bab-d20d-43f1-a48e-4bf555c47039"
+					(reference "U2")
+					(unit 1)
+				)

Commit message: schematic complete
Parts:
- removed AE1: Antenna, symbol Device:Antenna
- removed C13, C14: 1.5pF, PCM_JLCPCB:C_0402, symbol PCM_JLCPCB-Capacitors:0402,1.5pF
- removed C15: 100pF, PCM_JLCPCB:C_0402, symbol PCM_JLCPCB-Capacitors:0402,100pF
- removed C6, C7, C8: 100nF, PCM_JLCPCB:C_0603, symbol PCM_JLCPCB-Capacitors:0603,100nF
- removed R15, R6, R7, R8, R9: 0Ω, PCM_JLCPCB:R_0603, symbol PCM_JLCPCB-Resistors:0603,0Ω
- removed U3: AMS1117, PCM_JLCPCB:SOT-223-3_L6.5-W3.4-P2.30-LS7.0-BR, symbol PCM_JLCPCB-Power:LDO, 3.3V, 1A
- added AE2: Antenna_Chip, Capacitor_SMD:C_1206_3216Metric, symbol Device:Antenna_Chip
- added C13: 100nF, PCM_JLCPCB:C_0603, symbol PCM_JLCPCB-Capacitors:0603,100nF
- added C17: 10uF, PCM_JLCPCB:C_0805, symbol PCM_JLCPCB-Capacitors:0805,10uF
- added D1: Green, PCM_JLCPCB:D_0805, symbol PCM_JLCPCB-Diodes:LED,0805,Green
- added D2: Red, PCM_JLCPCB:D_0805, symbol PCM_JLCPCB-Diodes:LED,0805,Red
- added J1: Conn_01x02_Pin, Connector_JST:JST_PH_B2B-PH-K_1x02_P2.00mm_Vertical, symbol Connector:Conn_01x02_Pin
- added J3: Conn_01x04_Pin, Connector_PinSocket_2.54mm:PinSocket_1x04_P2.54mm_Vertical, symbol Connector:Conn_01x04_Pin
- added J4: Conn_01x02_Pin, symbol Connector:Conn_01x02_Pin
- added R10: 510Ω, PCM_JLCPCB:R_0603, symbol PCM_JLCPCB-Resistors:0603,510Ω
- added R11: 360Ω, PCM_JLCPCB:R_0603, symbol PCM_JLCPCB-Resistors:0603,360Ω
- added R12, R13, R14, R15: 10kΩ, PCM_JLCPCB:R_0805, symbol PCM_JLCPCB-Resistors:0805,10kΩ
- added TP1, TP2, TP3, TP4, TP5, TP6, TP7, TP8, TP9: TestPoint, TestPoint:TestPoint_Pad_D1.0mm, symbol Connector:TestPoint
- added U4: TP4057, PCM_JLCPCB:SOT-23-6_L2.9-W1.6-P0.95-LS2.8-BL, symbol PCM_JLCPCB-Power:Battery, Li-Ion, 0.5A, TP4057
- added U5: MCP1700x-330xxTT, Package_TO_SOT_SMD:SOT-23, symbol Regulator_Linear:MCP1700x-330xxTT
Connections:
- net CS_ACC is gone; now on net SDA: R5.1
- net MISO is gone; now on net SCK: R4.1
- net +3V3: now also U2.3 (VDD), C13.1, J3.2 (Pin_2), R13.1, R14.1, U5.2 (VO)
- net GND: now also U2.4 (SDA/PWM), AE2.1 (FEED), C13.2, C17.2, J1.2 (Pin_2), J3.1 (Pin_1), R12.1, R15.2, U4.2 (GND), U5.1 (GND)
- net SCK: now also U2.1 (SCL/Vz), J3.3 (Pin_3)
- net at U1.15 (GPIO9): now also J4.1 (Pin_1), TP4.1
- net at U1.8 (GPIO3): now also R5.2
- net at U1.6 (GPIO2): now also R13.2, TP5.1; no longer R4.2
- net at U1.16 (GPIO10): now also R4.2; no longer R5.2
- net SDA: now reaches U2.4 (SDA/PWM)
- net SDA: now also J3.4 (Pin_4)
- net at U1.1 (LNA_IN): now also AE2.2 (PCB_Trace)
- net at R1.1: now also TP1.1
- net at U1.14 (GPIO8): now also R14.2, TP3.1
- net at U1.21 (SPICS0): now also TP9.1
- net at U1.22 (SPICLK): now also TP8.1
- net at U1.23 (SPID): now also TP7.1
- net at U1.24 (SPIQ): now also TP6.1
- net at U1.27 (U0RXD): now also TP2.1
- net +5V renamed VBAT
- net VBAT: now also J1.1 (Pin_1), U4.3 (BAT), U5.3 (VI); no longer R32.2
- new net: D2.2, R10.2
- new net: D2.1, U4.1 (CHRG)
- new net: D1.1, U4.5 (STDBY)
- new net: R12.2, U4.6 (PROG)
- new net: J4.2 (Pin_2), R15.1
- new net: D1.2, R11.2
- new net VBUS: C17.1, R10.1, R11.1, R32.2, U4.4 (VCC)
Other:
- note added: "100mA CC"
- note added: "DCI variant 3V gradient compensated"
- moved on the sheet: C1, C16, C2, C3, C4, C5, C9, FB1, R17, U2

Commit message: schematic complete
Parts:
- removed C1, C12, C13, C2, C3, C4: 100nF, PCM_JLCPCB:C_0603, symbol PCM_JLCPCB-Capacitors:0603,100nF
- removed C16, C17, C5: 10uF, PCM_JLCPCB:C_0805, symbol PCM_JLCPCB-Capacitors:0805,10uF
- removed C9: 1uF, PCM_JLCPCB:C_0603, symbol PCM_JLCPCB-Capacitors:0603,1uF
- removed J4: Conn_01x02_Pin, symbol Connector:Conn_01x02_Pin
- removed R1: 470Ω, PCM_JLCPCB:R_0603, symbol PCM_JLCPCB-Resistors:0603,470Ω
- removed R10: 510Ω, PCM_JLCPCB:R_0603, symbol PCM_JLCPCB-Resistors:0603,510Ω
- removed R11: 360Ω, PCM_JLCPCB:R_0603, symbol PCM_JLCPCB-Resistors:0603,360Ω
- removed R12, R13, R14, R15: 10kΩ, PCM_JLCPCB:R_0805, symbol PCM_JLCPCB-Resistors:0805,10kΩ
- removed R3: 1kΩ, PCM_JLCPCB:R_0603, symbol PCM_JLCPCB-Resistors:0603,1kΩ
- removed R32, R4, R5: 0Ω, PCM_JLCPCB:R_0603, symbol PCM_JLCPCB-Resistors:0603,0Ω
- removed R33, R34: 5.1kΩ, PCM_JLCPCB:R_0603, symbol PCM_JLCPCB-Resistors:0603,5.1kΩ
- removed TP6, TP7, TP8, TP9: TestPoint, TestPoint:TestPoint_Pad_D1.0mm, symbol Connector:TestPoint
- added C1, C3, C4, C5: 10uF, PCM_JLCPCB:C_0603, symbol PCM_JLCPCB-Capacitors:0603,10uF,(2)
- added C15, C19, C20, C21, C22, C6: 100nF, PCM_JLCPCB:C_0402, symbol PCM_JLCPCB-Capacitors:0402,100nF
- added C2: 1uF, PCM_JLCPCB:C_0402, symbol PCM_JLCPCB-Capacitors:0402,1uF
- added D3: 1N4001W, PCM_JLCPCB:D_SOD-123FL, symbol PCM_JLCPCB-Diodes:General,1N4001W
- added J5, J6: Conn_01x02_Pin, TestPoint:TestPoint_2Pads_Pitch2.54mm_Drill0.8mm, symbol Connector:Conn_01x02_Pin
- added Q1: HJ8205, PCM_JLCPCB:SOT-23-6_L2.9-W1.6-P0.95-LS2.8-BR, symbol PCM_JLCPCB-Transistor-Packages:NMOS, 2 Channel, HJ8205
- added Q2: HL2305, PCM_JLCPCB:Q_SOT-23, symbol PCM_JLCPCB-Transistors:PMOS,HL2305
- added R1: 510Ω, PCM_JLCPCB:R_0402, symbol PCM_JLCPCB-Resistors:0402,510Ω
- added R10: 1kΩ, PCM_JLCPCB:R_0402, symbol PCM_JLCPCB-Resistors:0402,1kΩ
- added R11, R12, R13, R5, R8: 10kΩ, PCM_JLCPCB:R_0402, symbol PCM_JLCPCB-Resistors:0402,10kΩ
- added R14, R15: 5.1kΩ, PCM_JLCPCB:R_0402, symbol PCM_JLCPCB-Resistors:0402,5.1kΩ
- added R18, R19, R20, R9: 0Ω, PCM_JLCPCB:R_0402, symbol PCM_JLCPCB-Resistors:0402,0Ω
- added R21, R22: 470Ω, PCM_JLCPCB:R_0402, symbol PCM_JLCPCB-Resistors:0402,470Ω
- added R3, R4: 4.7kΩ, PCM_JLCPCB:R_0402, symbol PCM_JLCPCB-Resistors:0402,4.7kΩ
- added R6: 330Ω, PCM_JLCPCB:R_0402, symbol PCM_JLCPCB-Resistors:0402,330Ω
- added R7: 2kΩ, PCM_JLCPCB:R_0402, symbol PCM_JLCPCB-Resistors:0402,2kΩ
- added U3: DW01A, Package_TO_SOT_SMD:SOT-23-6, symbol Battery_Management:DW01A
- J1: footprint Connector_JST:JST_PH_B2B-PH-K_1x02_P2.00mm_Vertical -> TestPoint:TestPoint_2Pads_Pitch2.54mm_Drill0.8mm
Connections:
- net +3V3: now also C19.1, C20.1, C21.1, C22.1, C4.1, C5.1, R10.2, R11.1, R13.1, R3.1, R4.1, R5.1
- net 3V3_FILT: now also C2.1
- net GND: now also C1.2, C15.2, C19.2, C2.2, C20.2, C21.2, C22.2, C3.2, C4.2, C5.2, J6.2 (Pin_2), Q1.3 (S2), R12.1, R14.2, R15.2, R7.2, R8.2, R9.2; no longer J1.2 (Pin_2)
- net SCK: now also R20.1, R4.2
- net SDA: now also U2.2 (SDA/PWM), R19.1, R3.2; no longer U2.4 (SDA/PWM)
- net VBAT: now also Q2.3 (D), R22.2; no longer U5.3 (VI)
- net VBUS: now also C3.1, D3.2, J6.1 (Pin_1), Q2.1 (G), R1.1, R18.2, R6.1, R8.1
- net at TP4.1, U1.15 (GPIO9): now also R11.2
- net at D2.2: now also R1.2
- net at TP5.1, U1.6 (GPIO2): now also R13.2
- net at TP3.1, U1.14 (GPIO8): now also R5.2
- net at U4.6 (PROG): now also R12.2
- net at J2.A4 (VBUS), J2.A9 (VBUS), J2.B4 (VBUS)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: now also R18.1
- net at J2.A5 (CC1): now also R14.1
- net at J2.B5 (CC2): now also R15.1
- net at U1.7 (CHIP_EN): now also C15.1, R10.1
- net at D1.2: now also R6.2
- net at TP1.1: now also R21.1
- net at U1.28 (U0TXD): now also R21.2
- net at U1.16 (GPIO10): now also R20.2
- net at U1.8 (GPIO3): now also R19.2
- new net: C6.1, R22.1, U3.5 (VCC)
- new net: R7.1, U3.2 (CS)
- new net: Q1.6 (G1), U3.1 (OD)
- new net: Q1.4 (G2), U3.3 (OC)
- new net: C6.2, J1.2 (Pin_2), Q1.1 (S1), R9.1, U3.6 (GND)
- new net: C1.1, J5.1 (Pin_1), U5.3 (VI)
- new net: D3.1, J5.2 (Pin_2), Q2.2 (S)
- new net: Q1.2 (D1/D2), Q1.5 (D1/D2)
Other:
- note added: "20.20mm"
- note added: "30deg"
- note added: "32.32mm to create 60deg V60 taper"
- note added: "9mm"
- note added: "Battery charger"
- note added: "Battery protection"
- note added: "Display"
- note added: "MLX90614 IR temp sensor"
- note added: "Power source selection and LDO"
- note added: "protection bypass"
- moved on the sheet: AE2, C10, C11, D1, D2, FB1, J2, J3, R17, R2, TP1, TP2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

Commit message: routing complete
Parts:
- removed Q1: HJ8205, PCM_JLCPCB:SOT-23-6_L2.9-W1.6-P0.95-LS2.8-BR, symbol PCM_JLCPCB-Transistor-Packages:NMOS, 2 Channel, HJ8205
- added J7, J8: Conn_01x02_Pin, TestPoint:TestPoint_2Pads_Pitch2.54mm_Drill0.8mm, symbol Connector:Conn_01x02_Pin
- added Q3: HJ8205, PCM_JLCPCB:SOT-23-6_L2.9-W1.6-P0.95-LS2.8-BR, symbol 0_MyLib:NMOS, 2 Channel, HJ8205
- added R23, R24: 10kΩ, PCM_JLCPCB:R_0402, symbol PCM_JLCPCB-Resistors:0402,10kΩ
- added TP6, TP7, TP8: TestPoint, TestPoint:TestPoint_Pad_D1.0mm, symbol Connector:TestPoint
Connections:
- net +3V3: now also R23.1, R24.1
- net GND: now also J7.2 (Pin_2), J8.2 (Pin_2), Q3.3 (S2), TP6.1, TP7.1, TP8.1; no longer AE2.1 (FEED)
- net at U3.1 (OD): now also Q3.6 (G1)
- net at U3.3 (OC): now also Q3.4 (G2)
- net at C6.2, J1.2 (Pin_2), R9.1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: now also Q3.1 (S1)
- net USB_ESP_P: now reaches R17.2, U1.26 (GPIO19/USB_D+)
- net USB_ESP_N: now reaches R16.2, U1.25 (GPIO18/USB_D-)
- net at U1.4 (GPIO0/XTAL_32K_P): now also J7.1 (Pin_1), R23.2
- net at U1.5 (GPIO1/XTAL_32K_N): now also J8.1 (Pin_1), R24.2
- new net: Q3.2 (D1/D2), Q3.5 (D1/D2)
- no-connect marks 0 -> 1
Other:
- note added: "Batt term"
- note added: "To PWR switch"
- moved on the sheet: J1

Commit message: release for fab
Parts:
- removed TP6: TestPoint, TestPoint:TestPoint_Pad_D1.0mm, symbol Connector:TestPoint
- AE2: LCSC (none) -> C127629
- J1, J5, J6, J7, J8, TP1, TP2, TP3, TP4, TP5, TP7, TP8, U2: now left out of the parts list
- J3: LCSC (none) -> C2718488; now left out of the parts list
- U3: LCSC (none) -> C18164398
- U5: LCSC (none) -> C39051
Changed lines of the file:
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@@
 	(wire
 		(pts
-			(xy 153.67 83.82) (xy 153.67 82.55)
-		)
-		(stroke
-			(width 0)
-			(type default)
-		)
-	)
-	(wire
-		(pts
 			(xy 67.31 123.19) (xy 67.31 125.73)
 		)
@@
 			)
 		)
+		(property "LCSC" "C18164398"
+			(at 54.61 41.91 0)
+			(hide yes)
+			(show_name no)
+			(do_not_autoplace no)
+			(effects
+				(font
+					(size 1.27 1.27)
+				)
+			)
+		)
 		(pin "4"
 		)
@@
 		(body_style 1)
 		(exclude_from_sim no)
-		(in_bom yes)
+		(in_bom no)
 		(on_board yes)
 		(in_pos_files yes)
@@
 		(body_style 1)
 		(exclude_from_sim no)
-		(in_bom yes)
+		(in_bom no)
 		(on_board yes)
 		(in_pos_files yes)
@@
 		(body_style 1)
 		(exclude_from_sim no)
-		(in_bom yes)
+		(in_bom no)
 		(on_board yes)
 		(in_pos_files yes)
@@
 		(body_style 1)
 		(exclude_from_sim no)
-		(in_bom yes)
+		(in_bom no)
 		(on_board yes)
 		(in_pos_files yes)
@@
 		(body_style 1)
 		(exclude_from_sim no)
-		(in_bom yes)
+		(in_bom no)
 		(on_board yes)
 		(in_pos_files yes)
@@
 		(body_style 1)
 		(exclude_from_sim no)
-		(in_bom yes)
+		(in_bom no)
 		(on_board yes)
 		(in_pos_files yes)
@@
 		(body_style 1)
 		(exclude_from_sim no)
-		(in_bom yes)
+		(in_bom no)
 		(on_board yes)
 		(in_pos_files yes)
@@
 		(body_style 1)
 		(exclude_from_sim no)
-		(in_bom yes)
+		(in_bom no)
 		(on_board yes)
 		(in_pos_files yes)
@@
 			)
 		)
+		(property "LCSC" "C2718488"
+			(at 241.3 120.65 0)
+			(hide yes)
+			(show_name no)
+			(do_not_autoplace no)
+			(effects
+				(font
+					(size 1.27 1.27)
+				)
+			)
+		)
 		(pin "2"
 		)
@@
 		(body_style 1)
 		(exclude_from_sim no)
-		(in_bom yes)
+		(in_bom no)
 		(on_board yes)
 		(in_pos_files yes)
@@
 		(body_style 1)
 		(exclude_from_sim no)
-		(in_bom yes)
+		(in_bom no)
 		(on_board yes)
 		(in_pos_files yes)
@@
 	)
 	(symbol
-		(lib_id "power:GND")
-		(at 153.67 83.82 0)
-		(unit 1)
-		(body_style 1)
-		(exclude_from_sim no)
-		(in_bom yes)
-		(on_board yes)
-		(in_pos_files yes)
-		(dnp no)
-		(fields_autoplaced yes)
-		(property "Reference" "#PWR041"
-			(at 153.67 90.17 0)
-			(hide yes)
-			(show_name no)
-			(do_not_autoplace no)
-			(effects
-				(font
-					(size 1.27 1.27)
-				)
-			)
-		)
-		(property "Value" "GND"
-			(at 153.67 88.9 0)
-			(hide yes)
-			(show_name no)
-			(do_not_autoplace no)
-			(effects
-				(font
-					(size 1.27 1.27)
-				)
-			)
-		)
-		(property "Footprint" ""
-			(at 153.67 83.82 0)
-			(hide yes)
-			(show_name no)
-			(do_not_autoplace no)
-			(effects
-				(font
-					(size 1.27 1.27)
-				)
-			)
-		)
-		(property "Datasheet" ""
-			(at 153.67 83.82 0)
-			(hide yes)
-			(show_name no)
-			(do_not_autoplace no)
-			(effects
-				(font
-					(size 1.27 1.27)
-				)
-			)
-		)
-		(property "Description" "Power symbol creates a global label with name \"GND\" , ground"
-			(at 153.67 83.82 0)
-			(hide yes)
-			(show_name no)
-			(do_not_autoplace no)
-			(effects
-				(font
-					(size 1.27 1.27)
-				)
-			)
-		)
-		(pin "1"
-		)
-		(instances
-			(project "IR coffee thermometer"
-				(path "/ed3d3bab-d20d-43f1-a48e-4bf555c47039"
-					(reference "#PWR041")
-					(unit 1)
-				)
-			)
-		)
-	)
-	(symbol
 		(lib_id "PCM_JLCPCB-Resistors:0402,0Ω")
 		(at 60.96 115.57 90)
@@
 		(body_style 1)
 		(exclude_from_sim no)
-		(in_bom yes)
+		(in_bom no)
 		(on_board yes)
 		(in_pos_files yes)
@@
 	)
 	(symbol
-		(lib_id "Connector:TestPoint")
-		(at 153.67 82.55 0)
-		(unit 1)
-		(body_style 1)
-		(exclude_from_sim no)
-		(in_bom yes)
-		(on_board yes)
-		(in_pos_files yes)
-		(dnp no)
-		(property "Reference" "TP6"
-			(at 153.67 74.93 90)
-			(show_name no)
-			(do_not_autoplace no)
-			(effects
-				(font
-					(size 1.27 1.27)
-				)
-			)
-		)
-		(property "Value" "TestPoint"
-			(at 156.21 79.248 90)
-			(hide yes)
-			(show_name no)
-			(do_not_autoplace no)
-			(effects
-				(font
-					(size 1.27 1.27)
-				)
-			)
-		)
-		(property "Footprint" "TestPoint:TestPoint_Pad_D1.0mm"
-			(at 158.75 82.55 0)
-			(hide yes)
-			(show_name no)
-			(do_not_autoplace no)
-			(effects
-				(font
-					(size 1.27 1.27)
-				)
-			)
-		)
-		(property "Datasheet" ""
-			(at 158.75 82.55 0)
-			(hide yes)
-			(show_name no)
-			(do_not_autoplace no)
-			(effects
-				(font
-					(size 1.27 1.27)
-				)
-			)
-		)
-		(property "Description" "test point"
-			(at 153.67 82.55 0)
-			(hide yes)
-			(show_name no)
-			(do_not_autoplace no)
-			(effects
-				(font
-					(size 1.27 1.27)
-				)
-			)
-		)
-		(pin "1"
-		)
-		(instances
-			(project "IR coffee thermometer"
-				(path "/ed3d3bab-d20d-43f1-a48e-4bf555c47039"
-					(reference "TP6")
-					(unit 1)
-				)
-			)
-		)
-	)
-	(symbol
 		(lib_id "power:+3V3")
 		(at 85.09 101.6 0)
@@
 		(body_style 1)
 		(exclude_from_sim no)
-		(in_bom yes)
+		(in_bom no)
 		(on_board yes)
 		(in_pos_files yes)
@@
 			)
 		)
+		(property "LCSC" "C127629"
+			(at 195.58 104.14 0)
+			(hide yes)
+			(show_name no)
+			(do_not_autoplace no)
+			(effects
+				(font
+					(size 1.27 1.27)
+				)
+			)
+		)
 		(pin "2"
 		)
@@
 			)
 		)
+		(property "LCSC" "C39051"
+			(at 198.12 45.72 0)
+			(hide yes)
+			(show_name no)
+			(do_not_autoplace no)
+			(effects
+				(font
+					(size 1.27 1.27)
+				)
+			)
+		)
 		(pin "2"
 		)
@@
 		(body_style 1)
 		(exclude_from_sim no)
-		(in_bom yes)
+		(in_bom no)
 		(on_board yes)
 		(in_pos_files yes)
@@
 		(body_style 1)
 		(exclude_from_sim no)
-		(in_bom yes)
+		(in_bom no)
 		(on_board yes)
 		(in_pos_files yes)
